Commit message: modif urdf

File: catkin_ws/src/motoman_copy/motoman_hc10_support/urdf/hc10.xacro (robot description, xacro)
@@ -7,3 +7,7 @@
   <xacro:include filename="$(find motoman_hc10_support)/urdf/hc10.control.xacro"/>
   <xacro:hc10_control arm_id=""/>
+  <xacro:include filename="$(find motoman_hc10_support)/urdf/kinect_macro.xacro" />
+  <xacro:motoman_hc10_kinect prefix=""/>
+  <xacro:include filename="$(find motoman_hc10_support)/urdf/robot2Kinect.xacro" />
+  <xacro:motoman_hc10_robot2Kinect prefix=""/>
 </robot>

File: catkin_ws/src/motoman_copy/motoman_hc10_support/urdf/hc10_macro.xacro (robot description, xacro)
@@ -73,5 +73,5 @@
       <collision>
         <geometry>
-          <mesh filename="package://motjoint_1_soman_hc10_support/meshes/hc10/collision/link_3_u.stl"/>
+          <mesh filename="package://motoman_hc10_support/meshes/hc10/collision/link_3_u.stl"/>
         </geometry>
       </collision>
@@ -131,5 +131,4 @@
       </collision>
     </link>
-    <link name="${prefix}tool0"/>
     <!-- end of link list -->
     <!-- joint list -->
@@ -186,9 +185,4 @@
       <limit lower="${radians(-180)}" upper="${radians(180)}" effort="31.36" velocity="${radians(250)}"/>
     </joint>
-    <joint name="${prefix}joint_6_t-tool0" type="fixed">
-      <origin xyz="0 0 -0.130" rpy="${pi} 0 0"/>
-      <parent link="${prefix}link_6_t"/>
-      <child link="${prefix}tool0"/>
-    </joint>
     <!-- end of joint list -->
     <!-- ROS base_link to Robot Manufacturer World Coordinates transform -->

Commit message: fix frame camera

File: catkin_ws/src/motoman_copy/motoman_hc10_support/urdf/hc10.xacro (robot description, xacro)
@@ -9,5 +9,3 @@
   <xacro:include filename="$(find motoman_hc10_support)/urdf/kinect_macro.xacro" />
   <xacro:motoman_hc10_kinect prefix=""/>
-  <xacro:include filename="$(find motoman_hc10_support)/urdf/robot2Kinect.xacro" />
-  <xacro:motoman_hc10_robot2Kinect prefix=""/>
 </robot>

File: catkin_ws/src/motoman_copy/motoman_hc10_support/urdf/hc10_macro.xacro (robot description, xacro)
@@ -131,4 +131,5 @@
       </collision>
     </link>
+    <link name="${prefix}tool0"/>
     <!-- end of link list -->
     <!-- joint list -->
@@ -185,12 +186,11 @@
       <limit lower="${radians(-180)}" upper="${radians(180)}" effort="31.36" velocity="${radians(250)}"/>
     </joint>
+    <joint name="${prefix}joint_6_t-tool0" type="fixed">
+      <origin xyz="0 0 -0.130" rpy="${pi} 0 0"/>
+      <parent link="${prefix}link_6_t"/>
+      <child link="${prefix}tool0"/>
+    </joint>
     <!-- end of joint list -->
     <!-- ROS base_link to Robot Manufacturer World Coordinates transform -->
-    <link name="${prefix}base" />
-    <joint name="${prefix}base_link-base" type="fixed">
-      <origin xyz="0 0 0.275" rpy="0 0 0"/>
-      <parent link="${prefix}base_link"/>
-      <child link="${prefix}base"/>
-    </joint>
   </xacro:macro>
 </robot>

File: catkin_ws/src/motoman_copy/motoman_hc10_support/urdf/kinect_macro.xacro (robot description, xacro)
@@ -4,7 +4,7 @@
     <xacro:include filename="$(find motoman_resources)/urdf/common_materials.xacro"/>
     <!-- link list -->
-    <link name="${prefix}tool0">
+    <link name="${prefix}camera_depth_frame">
       <inertial>
-        <origin xyz="0 0.06 -0.160" rpy="${pi} ${pi/2} ${pi/2}"/>
+        <origin xyz="0 0 0" rpy="0 0 0"/>
         <mass value="0.1"/>
         <inertia ixx="0.03" ixy="0.03" ixz="0.03" iyy="0.0" iyz="0.0" izz="00"/>
@@ -23,5 +23,10 @@
     </link>
     <!-- end of link list -->
-    <gazebo reference="camera_depth_frame">
+    <joint name="${prefix}tool0_t_cam" type="fixed">
+      <origin xyz="0 -0.06 0.05" rpy="0 ${-pi/2} ${-pi/2}"/>
+      <parent link="${prefix}tool0"/>
+      <child link="${prefix}camera_depth_frame"/>
+    </joint>
+    <gazebo reference="${prefix}camera_depth_frame">
     <sensor name="kinect_camera" type="depth">
         <update_rate>20</update_rate>

File: catkin_ws/src/motoman_copy/motoman_hc10_support/urdf/model_hc10.urdf (robot description, URDF)
Before this commit: robot motoman_hc10, 10 links, 9 joints
Links:
- link tool0: mass None -> 0.1; geometry collision mesh filename=package://motoman_hc10_support/meshes/hc10/collision/kinect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; visual mesh filename=package://motoman_hc10_support/meshes/hc10/visual/kinect.dae
Joints:
- joint joint_6_t-tool0: origin xyz=0 0 -0.130 rpy=3.141592653589793 0 0 -> xyz=0 0.06 -0.160 rpy=3.141592653589793 1.5707963267948966 1.5707963267948966
