Commit message: modif urdf

File: catkin_ws/src/motoman_copy/motoman_hc10_support/urdf/hc10_macro.xacro (robot description, xacro)
@@ -131,5 +131,4 @@
       </collision>
     </link>
-    <link name="${prefix}tool0"/>
     <!-- end of link list -->
     <!-- joint list -->
@@ -186,9 +185,4 @@
       <limit lower="${radians(-180)}" upper="${radians(180)}" effort="31.36" velocity="${radians(250)}"/>
     </joint>
-    <joint name="${prefix}joint_6_t-tool0" type="fixed">
-      <origin xyz="0 0 -0.130" rpy="${pi} 0 0"/>
-      <parent link="${prefix}link_6_t"/>
-      <child link="${prefix}tool0"/>
-    </joint>
     <!-- end of joint list -->
     <!-- ROS base_link to Robot Manufacturer World Coordinates transform -->

Commit message: fix frame camera

File: catkin_ws/src/motoman_copy/motoman_hc10_support/urdf/hc10_macro.xacro (robot description, xacro)
@@ -131,4 +131,5 @@
       </collision>
     </link>
+    <link name="${prefix}tool0"/>
     <!-- end of link list -->
     <!-- joint list -->
@@ -185,4 +186,9 @@
       <limit lower="${radians(-180)}" upper="${radians(180)}" effort="31.36" velocity="${radians(250)}"/>
     </joint>
+    <joint name="${prefix}joint_6_t-tool0" type="fixed">
+      <origin xyz="0 0 -0.130" rpy="${pi} 0 0"/>
+      <parent link="${prefix}link_6_t"/>
+      <child link="${prefix}tool0"/>
+    </joint>
     <!-- end of joint list -->
     <!-- ROS base_link to Robot Manufacturer World Coordinates transform -->

File: catkin_ws/src/motoman_copy/motoman_hc10_support/urdf/model_hc10.urdf (robot description, URDF)
Before this commit: robot motoman_hc10, 9 links, 8 joints
Links:
- removed link tool0
Joints:
- removed joint joint_6_t-tool0
