Commit message: add sensor link and add publisher

File: catkin_ws/src/motoman_copy/motoman_hc10_support/urdf/kinect_macro.xacro (robot description, xacro)
@@ -22,4 +22,5 @@
       </collision>
     </link>
+    <link name="camera_depth_optical_frame"/>
     <!-- end of link list -->
     <joint name="${prefix}tool0_t_cam" type="fixed">
@@ -27,4 +28,9 @@
       <parent link="${prefix}tool0"/>
       <child link="${prefix}camera_depth_frame"/>
+    </joint>
+    <joint name="${prefix}cam_t_optical" type="fixed">
+      <origin xyz="0 0 0" rpy=" ${-pi/2} 0 ${-pi/2}"/>
+      <parent link="${prefix}camera_depth_frame"/>
+      <child link="camera_depth_optical_frame"/>
     </joint>
     <gazebo reference="${prefix}camera_depth_frame">

File: catkin_ws/src/motoman_copy/motoman_hc10_support/urdf/model_hc10.urdf (robot description, URDF)
Before this commit: robot motoman_hc10, 10 links, 9 joints
Links:
- removed link base
- added link camera_depth_frame, mass 0.1; collision mesh filename=package://motoman_hc10_support/meshes/hc10/collision/kinect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; visual mesh filename=package://motoman_hc10_support/meshes/hc10/visual/kinect.dae
- added link camera_depth_optical_frame
- link tool0: mass 0.1 -> None; geometry 
Joints:
- removed joint base_link-base
- added joint cam_t_optical: type fixed, parent camera_depth_frame, child camera_depth_optical_frame, origin xyz=0 -0.06 0.05 rpy=0 -1.5707963267948966 -1.5707963267948966
- added joint tool0_t_cam: type fixed, parent tool0, child camera_depth_frame, origin xyz=0 -0.06 0.05 rpy=0 -1.5707963267948966 -1.5707963267948966
- joint joint_6_t-tool0: origin xyz=0 0.06 -0.160 rpy=3.141592653589793 1.5707963267948966 1.5707963267948966 -> xyz=0 0 -0.130 rpy=3.141592653589793 0 0
