Commit message: add sensor link and add publisher

File: catkin_ws/src/motoman_copy/motoman_hc10_support/urdf/model_hc10.urdf (robot description, URDF)
Before this commit: robot motoman_hc10, 8 links, 7 joints
Links:
- added link camera_depth_frame, mass 0.1; collision mesh filename=package://motoman_hc10_support/meshes/hc10/collision/kinect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; visual mesh filename=package://motoman_hc10_support/meshes/hc10/visual/kinect.dae
- added link camera_depth_optical_frame
- added link tool0
Joints:
- added joint cam_t_optical: type fixed, parent camera_depth_frame, child camera_depth_optical_frame, origin xyz=0 -0.06 0.05 rpy=0 -1.5707963267948966 -1.5707963267948966
- added joint joint_6_t-tool0: type fixed, parent link_6_t, child tool0, origin xyz=0 0 -0.130 rpy=3.141592653589793 0 0
- added joint tool0_t_cam: type fixed, parent tool0, child camera_depth_frame, origin xyz=0 -0.06 0.05 rpy=0 -1.5707963267948966 -1.5707963267948966
